File: pcb/terrarium/terrarium.kicad_pcb (KiCad board)
At the start: 2 copper layers, 10 parts

Commit message: pcb v1.0
Parts:
- i2c LCD: renamed from i2c2
- i2c RTC: renamed from i2c1
- moved relay2 32.8 mm to (85.3, 84.3)
- moved relay1 19.1 mm to (111.8, 83.8)
Routing:
- net VCC: track 103.6 -> 174.6 mm
- net G5: track 0.00 -> 48.7 mm
- net G4: track 0.00 -> 36.4 mm
- net 3v3: track 0.00 -> 26.5 mm
- net (no net): vias 0 -> 4
- added copper zone on B.Cu, net GND
Other:
- board text added: "terrarium controller v1.0 github.com/brushknight/terrarium"

Commit message: updated PCB
Parts:
- added External Power: Conn_01x03, Connector_PinHeader_2.54mm:PinHeader_1x03_P2.54mm_Vertical, F.Cu at (48.3, 62.2)
- i2c1: renamed from i2c RTC
- i2c2: renamed from i2c LCD
- moved relay2 5.11 mm to (80.3, 83.8), turned to 90 degrees
- moved relay1 5.08 mm to (106.7, 83.8), turned to 90 degrees
Routing:
- net VCC: track 174.6 -> 232.0 mm
- net 3v3: track 26.5 -> 51.4 mm
- net G4: track 36.4 -> 35.3 mm
- net G5: track 48.7 -> 49.5 mm
Other:
- board text added: "3v3"
- board text added: "G16"
- board text added: "G17"
- board text added: "G18"
- board text added: "G19"
- board text added: "G21"
- board text added: "G22"
- board text added: "G4"
- board text added: "G5"
- board text added: "GND"
- board text added: "LCD"
- board text added: "RTC"
- board text added: "Relay 1"
- board text added: "Relay 2"
- board text added: "SCL"
- board text added: "SDA"
- board text added: "Signal"
- board text added: "VCC"

Commit message: add support for old pcb, add final changes to pcb
Parts:
- added G***: LOGO, logo_fp:snake_logo, F.Cu at (51.3, 39.1)
- added i2c3: Extra_5v, Connector_PinHeader_2.54mm:PinHeader_1x04_P2.54mm_Vertical, F.Cu at (66.0, 57.1)
- added i2c4: Extra_3v3, Connector_PinHeader_2.54mm:PinHeader_1x04_P2.54mm_Vertical, F.Cu at (66.0, 62.0)
- added rxtx1: Conn_01x02, Connector_PinSocket_2.54mm:PinSocket_1x02_P2.54mm_Vertical, F.Cu at (66.0, 40.6)
- ExternalPower1: renamed from External Power
- moved temp1 10.7 mm to (117.6, 34.3)
- moved temp2 10.7 mm to (104.9, 34.3)
- moved temp3 10.7 mm to (90.9, 34.3)
- moved temp4 10.7 mm to (77.0, 34.3)
- moved i2c1 7.62 mm to (66.0, 74.9), turned to 270 degrees
- moved i2c2 7.62 mm to (66.0, 49.5), turned to 270 degrees
- moved relay2 0.76 mm to (79.5, 83.8)
Connections:
- esp32-left1 pad 15: Net-(esp32-left1-Pad15) -> RX
- esp32-left1 pad 16: Net-(esp32-left1-Pad16) -> TX
Routing:
- net VCC: track 232.0 -> 272.3 mm
- net RX: track 0.00 -> 31.2 mm
- net TX: track 0.00 -> 30.4 mm
- net 3v3: track 51.4 -> 72.7 mm
- net G19: track 20.9 -> 33.0 mm
- net G18: track 11.7 -> 23.1 mm
- net SCL: track 47.8 -> 55.4 mm
- net G17: track 12.3 -> 17.0 mm
- net G16: track 20.9 -> 17.7 mm
- net SDA: track 59.9 -> 61.0 mm
Other:
- board text added: "External Power"
- board text added: "RX"
- board text added: "TX"
- board text added: "i2c BUS"
- board text added: "temp 1"
- board text added: "temp 2"
- board text added: "temp 3"
- board text added: "temp 4"
- board text added: "tx/rx"
- board text removed: "Relay 2"

Commit message: add gerber files
Other:
- board outline added: 90 x 90 mm
- board text added: "JLCJLCJLCJLC"

Commit message: wip: relay scheme
Parts:
- added K1: SANYOU_SRD_Form_C, Relay_THT:Relay_SPDT_SANYOU_SRD_Series_Form_C, F.Cu at (112.8, 90.4)
Connections:
- net 3v3 renamed +3V3
- net VCC renamed +5V
Other:
- board text added: "Relay 2"

Commit message: wip: re-do pcb, add relay
Parts:
- removed K1: SANYOU_SRD_Form_C, Relay_THT:Relay_SPDT_SANYOU_SRD_Series_Form_C
- added D1: 1N47xxA, Diode_THT:D_DO-41_SOD81_P10.16mm_Horizontal, F.Cu at (129.5, 126.4)
- added D5: ACTIVE, LED_THT:LED_D3.0mm_Clear, F.Cu at (80.0, 135.3)
- added J3: Screw_Terminal_01x03, Connector_PinSocket_2.54mm:PinSocket_1x03_P2.54mm_Vertical, F.Cu at (126.4, 160.7)
- added K3: SANYOU_SRD_Form_C, Relay_THT:Relay_SPDT_SANYOU_SRD_Series_Form_C, F.Cu at (123.8, 139.0)
- added Q2: MMBT3904, Package_TO_SOT_SMD:SOT-23, F.Cu at (97.4, 149.9)
- added R5: R_Small, Resistor_THT:R_Axial_DIN0204_L3.6mm_D1.6mm_P2.54mm_Vertical, F.Cu at (100.3, 118.1)
- added R6: R_Small, Resistor_THT:R_Axial_DIN0204_L3.6mm_D1.6mm_P2.54mm_Vertical, F.Cu at (99.1, 141.0)
- added U2: MOC3020M, Package_DIP:DIP-6_W7.62mm, F.Cu at (91.4, 127.6)
- moved temp4 10.7 mm to (87.6, 33.0), turned to 180 degrees
- moved temp3 6.97 mm to (97.8, 33.0), turned to 180 degrees
- moved temp2 2.73 mm to (107.3, 33.0), turned to 180 degrees
- moved temp1 1.48 mm to (116.8, 33.0), turned to 180 degrees
Routing:
- net +5V: track 272.3 -> 228.5 mm
- net G19: track 33.0 -> 0.00 mm
- net G18: track 23.1 -> 0.00 mm
- net G16: track 17.7 -> 0.00 mm
- net G17: track 17.0 -> 0.00 mm
Other:
- board text added: "5v"

Commit message: wip: update pcb
Parts:
- removed D5: ACTIVE, LED_THT:LED_D3.0mm_Clear
- removed J3: Screw_Terminal_01x03, Connector_PinSocket_2.54mm:PinSocket_1x03_P2.54mm_Vertical
- removed Q2: MMBT3904, Package_TO_SOT_SMD:SOT-23
- removed R5: R_Small, Resistor_THT:R_Axial_DIN0204_L3.6mm_D1.6mm_P2.54mm_Vertical
- removed U2: MOC3020M, Package_DIP:DIP-6_W7.62mm
- added D2: 1N47xxA, Diode_THT:D_DO-41_SOD81_P7.62mm_Horizontal, F.Cu at (96.0, 100.1)
- added LED1: ACTIVE, LED_THT:LED_D3.0mm_Clear, F.Cu at (110.7, 72.1)
- added LED2: ACTIVE, LED_THT:LED_D3.0mm_Clear, F.Cu at (83.8, 72.1)
- added OC1: MOC3020M, Package_DIP:DIP-6_W7.62mm, F.Cu at (123.4, 76.7)
- added OC2: MOC3020M, Package_DIP:DIP-6_W7.62mm, F.Cu at (96.5, 76.7)
- added R1: R_Small, Resistor_THT:R_Axial_DIN0204_L3.6mm_D1.6mm_P2.54mm_Vertical, F.Cu at (113.3, 78.7)
- added R3: R_Small, Resistor_THT:R_Axial_DIN0204_L3.6mm_D1.6mm_P2.54mm_Vertical, F.Cu at (86.4, 78.7)
- added R4: R_Small, Resistor_THT:R_Axial_DIN0204_L3.6mm_D1.6mm_P2.54mm_Vertical, F.Cu at (75.8, 82.5)
- added RE2: SANYOU_SRD_Form_C, Relay_THT:Relay_SPDT_SANYOU_SRD_Series_Form_C, F.Cu at (85.1, 88.9)
- added S1: Screw_Terminal_01x03, Connector_PinSocket_2.54mm:PinSocket_1x03_P2.54mm_Vertical, F.Cu at (114.3, 110.2)
- added S2: Screw_Terminal_01x03, Connector_PinSocket_2.54mm:PinSocket_1x03_P2.54mm_Vertical, F.Cu at (87.6, 110.5)
- added TR1: MMBT3904, Package_TO_SOT_THT:TO-92, F.Cu at (104.6, 73.7)
- added TR2: MMBT3904, Package_TO_SOT_THT:TO-92, F.Cu at (77.5, 75.2)
- added temp5: 4, Connector_JST:JST_XH_B3B-XH-AM_1x03_P2.50mm_Vertical, F.Cu at (108.6, 33.7)
- added temp6: 4, Connector_JST:JST_XH_B3B-XH-AM_1x03_P2.50mm_Vertical, F.Cu at (118.1, 33.7)
- D1: footprint Diode_THT:D_DO-41_SOD81_P10.16mm_Horizontal -> Diode_THT:D_DO-41_SOD81_P7.62mm_Horizontal
- i2c2: footprint Connector_PinHeader_2.54mm:PinHeader_1x04_P2.54mm_Vertical -> Connector_JST:JST_XH_B4B-XH-AM_1x04_P2.50mm_Vertical
- temp1, temp2, temp3, temp4: footprint Connector_PinHeader_2.54mm:PinHeader_1x03_P2.54mm_Vertical -> Connector_JST:JST_XH_B3B-XH-AM_1x03_P2.50mm_Vertical
- moved R2 58.2 mm to (101.6, 82.8), turned to 270 degrees
- moved RE1 51.6 mm to (111.8, 88.9)
- moved D1 27.2 mm to (122.4, 100.1), turned to 90 degrees
- moved temp1 17.8 mm to (99.1, 33.7), turned to 90 degrees
- moved temp2 17.8 mm to (89.5, 33.7), turned to 90 degrees
- moved temp3 17.8 mm to (80.0, 33.7), turned to 90 degrees
- moved temp4 17.2 mm to (70.5, 33.7), turned to 90 degrees
- moved esp32-right1 8.64 mm to (127.0, 66.3)
- moved esp32-left1 8.64 mm to (127.0, 40.9)
- moved G*** 7.22 mm to (55.4, 33.1), turned to 0 degrees
- moved rxtx1 6.36 mm to (72.4, 40.9), turned to 90 degrees
- moved relay2 0.76 mm to (80.3, 83.8)
- moved i2c2 0.25 mm to (66.0, 49.8), turned to 180 degrees
- renumbered R6 to R2, K3 to RE1
Connections:
- esp32-left1 pad 4: Net-(esp32-left1-Pad4) -> G15
- esp32-left1 pad 5: Net-(esp32-left1-Pad5) -> G2
Routing:
- net +5V: track 228.5 -> 279.2 mm
- net Net-(D1-Pad2): track 0.00 -> 40.3 mm
- net Net-(D2-Pad2): track 0.00 -> 37.3 mm
- net G19: track 0.00 -> 33.4 mm
- net G18: track 0.00 -> 25.6 mm
- net Net-(RE1-Pad1): track 0.00 -> 22.1 mm
- net Net-(RE2-Pad1): track 0.00 -> 21.6 mm
- net G17: track 0.00 -> 21.2 mm
- net Net-(OC1-Pad4): track 0.00 -> 18.0 mm
- net Net-(OC2-Pad4): track 0.00 -> 16.6 mm
- net G2: track 0.00 -> 15.5 mm
- net +3V3: track 72.7 -> 57.4 mm
- net TX: track 30.4 -> 16.0 mm
- net G16: track 0.00 -> 14.2 mm
- net G15: track 0.00 -> 12.6 mm
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Other:
- board text added: "G"
- board text added: "G15"
- board text added: "G2"
- board text added: "S"
- board text added: "terrarium controller v2.0 github.com/brushknight/terrarium"
- board text removed: "Relay 1"
- board text removed: "Relay 2"
- board text removed: "Signal"
- board text removed: "VCC"
- board text removed: "temp 1"
- board text removed: "temp 2"
- board text removed: "temp 3"
- board text removed: "temp 4"
- board text removed: "terrarium controller v1.0 github.com/brushknight/terrarium"

Commit message: wip: pcb relay design
Parts:
- removed OC1, OC2: MOC3020M, Package_DIP:DIP-6_W7.62mm
- S1, S2: footprint Connector_PinSocket_2.54mm:PinSocket_1x03_P2.54mm_Vertical -> TerminalBlock:TerminalBlock_bornier-3_P5.08mm
- moved TR1 17.4 mm to (121.9, 71.6), turned to 0 degrees
- moved TR2 16.6 mm to (94.0, 73.2), turned to 0 degrees
- moved R2 15.0 mm to (115.6, 77.5), turned to 0 degrees
- moved R4 14.3 mm to (86.6, 73.2), turned to 0 degrees
- moved R3 12.8 mm to (74.4, 83.3), turned to 0 degrees
- moved S2 9.25 mm to (90.2, 119.4), turned to 180 degrees
- moved LED2 7.91 mm to (75.9, 72.9)
- moved LED1 7.12 mm to (103.6, 71.9)
- moved R1 6.12 mm to (113.8, 72.6), turned to 0 degrees
- moved RE1 5.14 mm to (112.5, 83.8)
- moved relay1 3.81 mm to (106.7, 80.0)
- moved relay2 3.81 mm to (80.3, 80.0)
- moved S1 3.64 mm to (117.6, 108.7), turned to 180 degrees
Connections:
- LED1 pad 1: GND -> Net-(LED1-Pad1)
- LED1 pad 2: Net-(LED1-Pad2) -> G4
- LED2 pad 1: GND -> Net-(LED2-Pad1)
- LED2 pad 2: Net-(LED2-Pad2) -> G5
- R1 pad 1: Net-(OC1-Pad1) -> Net-(LED1-Pad1)
- R1 pad 2: G4 -> Net-(R1-Pad2)
- R2 pad 1: Net-(R2-Pad1) -> GND
- R2 pad 2: Net-(OC1-Pad4) -> Net-(R2-Pad2)
- R3 pad 1: Net-(OC2-Pad1) -> Net-(LED2-Pad1)
- R3 pad 2: G5 -> Net-(R3-Pad2)
- R4 pad 1: Net-(R4-Pad1) -> GND
- R4 pad 2: Net-(OC2-Pad4) -> Net-(R4-Pad2)
- TR1 pad 1: Net-(R2-Pad1) -> Net-(R1-Pad2)
- TR1 pad 2: GND -> Net-(R2-Pad2)
- TR2 pad 1: Net-(R4-Pad1) -> Net-(R3-Pad2)
- TR2 pad 2: GND -> Net-(R4-Pad2)
Routing:
- net Net-(OC1-Pad4): track 18.0 -> 0.00 mm
- net Net-(D2-Pad2): track 37.3 -> 19.8 mm
- net Net-(OC2-Pad4): track 16.6 -> 0.00 mm
- net Net-(OC2-Pad1): track 11.0 -> 0.00 mm
- net Net-(OC1-Pad1): track 11.0 -> 0.00 mm
- net Net-(R2-Pad1): track 10.4 -> 0.00 mm
- net Net-(LED2-Pad2): track 9.51 -> 0.00 mm
- net Net-(LED1-Pad2): track 9.51 -> 0.00 mm
- net Net-(R4-Pad1): track 8.05 -> 0.00 mm
