File: pcb/terrarium/terrarium.kicad_pcb (KiCad board)
At the start: 2 copper layers, 90 x 90 mm, 31 parts

Commit message: wip: finish with pcb layout
Parts:
- moved R3 15.6 mm to (85.9, 72.6)
- moved rxtx1 14.6 mm to (57.8, 40.4)
- moved D1 11.8 mm to (122.6, 88.3), turned to 270 degrees
- moved D2 11.7 mm to (95.5, 88.4), turned to 270 degrees
- moved S2 10.7 mm to (90.2, 108.7)
- moved R4 8.59 mm to (91.4, 80.3), turned to 90 degrees
- moved LED1 5.61 mm to (109.2, 72.4), turned to 180 degrees
- moved LED2 5.09 mm to (81.0, 72.6), turned to 180 degrees
- moved RE2 5.08 mm to (85.1, 83.8)
- moved R2 4.07 mm to (118.7, 80.0), turned to 90 degrees
- moved esp32-left1 3.81 mm to (123.2, 40.9)
- moved esp32-right1 3.81 mm to (123.2, 66.3)
- moved TR1 1.63 mm to (120.7, 72.6)
- moved R1 0.51 mm to (113.3, 72.6)
- moved TR2 0.51 mm to (94.0, 72.6)
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Routing:
- net +5V: track 279.2 -> 255.5 mm
- net Net-(D2-Pad2): track 19.8 -> 41.8 mm
- net TX: track 16.0 -> 26.0 mm
- net RX: track 21.8 -> 31.5 mm
- net Net-(R4-Pad2): track 0.00 -> 7.93 mm
- net Net-(R2-Pad2): track 0.00 -> 7.41 mm
- net G5: track 57.2 -> 51.0 mm
- net Net-(R3-Pad2): track 0.00 -> 5.59 mm
- net Net-(R1-Pad2): track 0.00 -> 4.95 mm
- net Net-(LED2-Pad1): track 0.00 -> 4.83 mm
- net G19: track 33.4 -> 28.8 mm
- net G4: track 46.3 -> 41.8 mm
- net Net-(LED1-Pad1): track 0.00 -> 4.32 mm
- net SDA: track 63.5 -> 59.7 mm
- net SCL: track 58.6 -> 54.8 mm
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
Commit message: wip: polish pcb
Parts:
- added H1: MountingHole, MountingHole:MountingHole_3.2mm_M3_DIN965_Pad, F.Cu at (127.0, 27.0)
- added H2: MountingHole, MountingHole:MountingHole_3.2mm_M3_DIN965_Pad, F.Cu at (45.0, 27.0)
- added H3: MountingHole, MountingHole:MountingHole_3.2mm_M3_DIN965_Pad, F.Cu at (45.0, 109.0)
- added H4: MountingHole, MountingHole:MountingHole_3.2mm_M3_DIN965_Pad, F.Cu at (127.0, 109.0)
- moved R4 5.68 mm to (96.5, 77.7), turned to 270 degrees
- moved R2 5.00 mm to (123.2, 77.7), turned to 270 degrees
Connections:
- R2 pad 1: GND -> Net-(R2-Pad1)
- R2 pad 2: Net-(R2-Pad2) -> Net-(D1-Pad2)
- R4 pad 1: GND -> Net-(R4-Pad1)
- R4 pad 2: Net-(R4-Pad2) -> Net-(D2-Pad2)
- TR1 pad 2: Net-(R2-Pad2) -> GND
- TR1 pad 3: Net-(D1-Pad2) -> Net-(R2-Pad1)
- TR2 pad 2: Net-(R4-Pad2) -> GND
- TR2 pad 3: Net-(D2-Pad2) -> Net-(R4-Pad1)
Routing:
- net Net-(R4-Pad2): track 7.93 -> 0.00 mm
- net Net-(D2-Pad2): track 41.8 -> 34.2 mm
- net Net-(D1-Pad2): track 40.8 -> 33.3 mm
- net Net-(R2-Pad2): track 7.41 -> 0.00 mm
- net Net-(R4-Pad1): track 0.00 -> 5.08 mm
- net Net-(R2-Pad1): track 0.00 -> 5.08 mm
- net +5V: track 255.5 -> 254.7 mm
- net (no net): vias 4 -> 0

Commit message: fix: gnd connectivity for TR1
Parts:
- renumbered temp6 to temp1, temp5 to temp2, temp1 to temp3, temp2 to temp4, temp3 to temp5, temp4 to temp6
Connections:
- S2 pad 1: Net-(RE2-Pad4) -> Net-(S2-Pad1)
Routing:
- net +5V: track 254.7 -> 257.0 mm

Commit message: fix: bug with RE2 terminal
Parts:
- renumbered temp3 to HT3, temp4 to HT4, temp5 to HT5
Connections:
- S2 pad 1: Net-(S2-Pad1) -> Net-(RE2-Pad4)
Other:
- board text added: "1"
- board text added: "2"
- board text added: "3"
- board text added: "4"
- board text added: "5"
- board text added: "6"
Changed lines of the file:
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@@
   (general
     (thickness 1.6)
-    (drawings 82)
+    (drawings 88)
     (tracks 137)
     (zones 0)
     (modules 35)
-    (nets 53)
+    (nets 52)
   )
   (page A4)
@@
   )
   (setup
-    (last_trace_width 0.4)
+    (last_trace_width 2)
     (user_trace_width 0.2)
     (user_trace_width 0.4)
@@
   (net 50 "Net-(R2-Pad1)")
   (net 51 "Net-(R4-Pad1)")
-  (net 52 "Net-(S2-Pad1)")
   (net_class Default "This is the default net class."
     (clearance 0.2)
@@
     (add_net "Net-(RE2-Pad3)")
     (add_net "Net-(RE2-Pad4)")
-    (add_net "Net-(S2-Pad1)")
     (add_net "Net-(esp32-left1-Pad1)")
     (add_net "Net-(esp32-left1-Pad18)")
@@
       (net 43 "Net-(RE2-Pad1)"))
     (pad 1 thru_hole rect (at 0 0 180) (size 3 3) (drill 1.52) (layers *.Cu *.Mask)
-      (net 52 "Net-(S2-Pad1)"))
+      (net 44 "Net-(RE2-Pad4)"))
     (model ${KISYS3DMOD}/TerminalBlock.3dshapes/TerminalBlock_bornier-3_P5.08mm.wrl
       (offset (xyz 5.079999923706055 0 0))
@@
     (descr "JST XH series connector, B3B-XH-AM, with boss (http://www.jst-mfg.com/product/pdf/eng/eXH.pdf), generated with kicad-footprint-generator")
     (tags "connector JST XH vertical boss")
-    (fp_text reference temp5 (at 8.89 0.635 180) (layer F.SilkS)
+    (fp_text reference HT5 (at 8.89 0.635 180) (layer F.SilkS)
       (effects (font (size 1 1) (thickness 0.15)))
     )
@@
     (descr "JST XH series connector, B3B-XH-AM, with boss (http://www.jst-mfg.com/product/pdf/eng/eXH.pdf), generated with kicad-footprint-generator")
     (tags "connector JST XH vertical boss")
-    (fp_text reference temp4 (at 8.81 0.635 180) (layer F.SilkS)
+    (fp_text reference HT4 (at 8.81 0.635 180) (layer F.SilkS)
       (effects (font (size 1 1) (thickness 0.15)))
     )
@@
     (descr "JST XH series connector, B3B-XH-AM, with boss (http://www.jst-mfg.com/product/pdf/eng/eXH.pdf), generated with kicad-footprint-generator")
     (tags "connector JST XH vertical boss")
-    (fp_text reference temp3 (at 8.89 0.635 180) (layer F.SilkS)
+    (fp_text reference HT3 (at 8.89 0.635 180) (layer F.SilkS)
       (effects (font (size 1 1) (thickness 0.15)))
     )
@@
     )
   )
+  (gr_text 1 (at 114.3 26) (layer F.SilkS)
+    (effects (font (size 2 2) (thickness 0.3)))
+  )
+  (gr_text 2 (at 104.775 26) (layer F.SilkS)
+    (effects (font (size 2 2) (thickness 0.3)))
+  )
+  (gr_text 3 (at 95.25 26) (layer F.SilkS)
+    (effects (font (size 2 2) (thickness 0.3)))
+  )
+  (gr_text 4 (at 85.598 26) (layer F.SilkS)
+    (effects (font (size 2 2) (thickness 0.3)))
+  )
+  (gr_text 5 (at 76.2 26) (layer F.SilkS)
+    (effects (font (size 2 2) (thickness 0.3)))
+  )
+  (gr_text 6 (at 66.675 26) (layer F.SilkS)
+    (effects (font (size 2 2) (thickness 0.3)))
+  )
   (gr_line (start 130.429 39.116) (end 124.968 39.116) (layer F.SilkS) (width 0.12))

Commit message: pcb: add ws2812b
Parts:
- added AD1: WS2812B, LED_SMD:LED_WS2812B_PLCC4_5.0x5.0mm_P3.2mm, F.Cu at (47.8, 45.7)
- added C1: 10pF, Capacitor_THT:C_Disc_D5.0mm_W2.5mm_P5.00mm, F.Cu at (45.2, 52.1)
Connections:
- esp32-left1 pad 18: Net-(esp32-left1-Pad18) -> G23
Routing:
- net G23: track 0.00 -> 31.1 mm, vias 0 -> 2
- net +5V: track 257.0 -> 272.9 mm
- net GND: track 0.00 -> 4.75 mm
Other:
- board text added: "Power"
- board text removed: "External Power"

Commit message: pcb minor changes
Parts:
- renumbered temp1 to HT1, temp2 to HT2, temp6 to HT6
Changed lines of the file:
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@@
-(kicad_pcb (version 20171130) (host pcbnew "(5.1.12-1-10_14)")
+(kicad_pcb (version 20171130) (host pcbnew 5.1.10-88a1d61d58~90~ubuntu21.04.1)
   (general
     (thickness 1.6)
     (drawings 88)
-    (tracks 152)
+    (tracks 154)
     (zones 0)
     (modules 37)
@@
   )
   (setup
-    (last_trace_width 0.4)
+    (last_trace_width 0.25)
     (user_trace_width 0.2)
     (user_trace_width 0.4)
@@
       (effects (font (size 1 1) (thickness 0.15)))
     )
-    (fp_text user %R (at 2.5 0) (layer F.Fab) hide
-      (effects (font (size 1 1) (thickness 0.15)))
-    )
     (fp_line (start 0 -1.25) (end 0 1.25) (layer F.Fab) (width 0.1))
     (fp_line (start 0 1.25) (end 5 1.25) (layer F.Fab) (width 0.1))
@@
     (fp_line (start 6.05 1.5) (end 6.05 -1.5) (layer F.CrtYd) (width 0.05))
     (fp_line (start 6.05 -1.5) (end -1.05 -1.5) (layer F.CrtYd) (width 0.05))
+    (fp_text user %R (at 2.5 0) (layer F.Fab) hide
+      (effects (font (size 1 1) (thickness 0.15)))
+    )
     (pad 2 thru_hole circle (at 5 0) (size 1.6 1.6) (drill 0.8) (layers *.Cu *.Mask)
       (net 1 GND))
@@
     )
     (fp_text value WS2812B (at 0 4) (layer F.Fab) hide
-      (effects (font (size 1 1) (thickness 0.15)))
-    )
-    (fp_text user %R (at 0 0) (layer F.Fab) hide
-      (effects (font (size 0.8 0.8) (thickness 0.15)))
-    )
-    (fp_text user 1 (at -4.15 -1.6) (layer F.SilkS) hide
       (effects (font (size 1 1) (thickness 0.15)))
     )
@@
     (fp_line (start 3.65 2.75) (end 3.65 1.6) (layer F.SilkS) (width 0.12))
     (fp_circle (center 0 0) (end 0 -2) (layer F.Fab) (width 0.1))
+    (fp_text user %R (at 0 0) (layer F.Fab) hide
+      (effects (font (size 0.8 0.8) (thickness 0.15)))
+    )
+    (fp_text user 1 (at -4.15 -1.6) (layer F.SilkS) hide
+      (effects (font (size 1 1) (thickness 0.15)))
+    )
     (pad 1 smd rect (at -2.45 -1.6) (size 1.5 1) (layers F.Cu F.Paste F.Mask)
       (net 34 +5V))
@@
     (descr "JST XH series connector, B3B-XH-AM, with boss (http://www.jst-mfg.com/product/pdf/eng/eXH.pdf), generated with kicad-footprint-generator")
     (tags "connector JST XH vertical boss")
-    (fp_text reference temp1 (at 8.89 0.635 180) (layer F.SilkS)
+    (fp_text reference HT1 (at 8.89 0.635 180) (layer F.SilkS)
       (effects (font (size 1 1) (thickness 0.15)))
     )
@@
     (descr "JST XH series connector, B3B-XH-AM, with boss (http://www.jst-mfg.com/product/pdf/eng/eXH.pdf), generated with kicad-footprint-generator")
     (tags "connector JST XH vertical boss")
-    (fp_text reference temp2 (at 8.89 0.635 180) (layer F.SilkS)
+    (fp_text reference HT2 (at 8.89 0.635 180) (layer F.SilkS)
       (effects (font (size 1 1) (thickness 0.15)))
     )
@@
     (descr "JST XH series connector, B3B-XH-AM, with boss (http://www.jst-mfg.com/product/pdf/eng/eXH.pdf), generated with kicad-footprint-generator")
     (tags "connector JST XH vertical boss")
-    (fp_text reference temp6 (at 8.89 0.635 180) (layer F.SilkS)
+    (fp_text reference HT6 (at 8.89 0.635 180) (layer F.SilkS)
       (effects (font (size 1 1) (thickness 0.15)))
     )
@@
   (segment (start 50.202 52.06) (end 50.212 52.07) (width 0.4) (layer F.Cu) (net 1))
   (segment (start 50.202 47.32) (end 50.202 52.06) (width 0.4) (layer F.Cu) (net 1))
-  (via (at 54.356 43.942) (size 0.8) (drill 0.4) (layers F.Cu B.Cu) (net 52))
-  (via (at 52.324 43.942) (size 0.8) (drill 0.4) (layers F.Cu B.Cu) (net 52))
   (segment (start 58.42 49.53) (end 58.42 57.15) (width 0.25) (layer F.Cu) (net 2))
   (segment (start 58.42 61.976) (end 58.42 57.15) (width 0.25) (layer F.Cu) (net 2))
@@
   (segment (start 83.312 39.116) (end 61.595 39.116) (width 0.25) (layer F.Cu) (net 31))
   (segment (start 85.09 40.894) (end 83.312 39.116) (width 0.25) (layer F.Cu) (net 31))
-  (segment (start 85.401991 38.665991) (end 59.505009 38.665991) (width 0.25) (layer F.Cu) (net 32))
   (segment (start 59.505009 38.665991) (end 57.785 40.386) (width 0.25) (layer F.Cu) (net 32))
   (segment (start 87.63 40.894) (end 85.401991 38.665991) (width 0.25) (layer F.Cu) (net 32))
+  (segment (start 59.505009 38.665991) (end 59.817 38.354) (width 0.25) (layer F.Cu) (net 32))
+  (segment (start 85.401991 38.665991) (end 85.09 38.354) (width 0.25) (layer F.Cu) (net 32))
+  (segment (start 85.09 38.354) (end 59.817 38.354) (width 0.25) (layer F.Cu) (net 32))
   (segment (start 63.5 74.93) (end 63.5 61.976) (width 0.4) (layer F.Cu) (net 33))
   (segment (start 63.5 72.39) (end 63.5 74.93) (width 0.4) (layer F.Cu) (net 33))
@@
   (segment (start 123.19 72.644) (end 123.19 77.724) (width 0.4) (layer F.Cu) (net 49))
   (segment (start 96.52 72.644) (end 96.52 77.724) (width 0.4) (layer F.Cu) (net 50))
+  (via (at 54.356 43.942) (size 0.8) (drill 0.4) (layers F.Cu B.Cu) (net 52))
+  (via (at 52.324 43.942) (size 0.8) (drill 0.4) (layers F.Cu B.Cu) (net 52))
   (segment (start 54.356 43.942) (end 52.324 43.942) (width 0.4) (layer B.Cu) (net 52))
   (segment (start 50.38 43.942) (end 50.202 44.12) (width 0.25) (layer F.Cu) (net 52))
