File: pcb/terrarium/terrarium.sch (KiCad schematic (older format))
At the start: 34 parts

Commit message: pcb: add ws2812b
Parts:
- added AD1: WS2812B, LED_SMD:LED_WS2812B_PLCC4_5.0x5.0mm_P3.2mm, symbol LED:WS2812B
- added C1: 10pF, Capacitor_THT:C_Disc_D5.0mm_W2.5mm_P5.00mm, symbol Device:C_Small
Connections:
- net +5V: now also AD1.1 (VDD), C1.1
- net GND: now also AD1.3 (VSS), C1.2
- net G23: now reaches esp32-left1.18 (Pin_18)
- net G23: now also AD1.4 (DIN)
- no-connect marks 32 -> 31
Changed lines of the file:
@@
 NoConn ~ 2050 4700
 NoConn ~ 2050 4800
-NoConn ~ 1200 4800
 NoConn ~ 4600 4700
 NoConn ~ 3800 4700
@@
 Daughter board relays
 Wire Notes Line
-	700  5750 3000 5750
-Wire Notes Line
-	3000 5750 3000 7100
-Wire Notes Line
-	3000 7100 700  7100
-Wire Notes Line
 	700  7100 700  5750
 Text Notes 700  5700 0    50   ~ 0
@@
 Wire Wire Line
 	8150 2650 9000 2650
+$Comp
+L LED:WS2812B AD1
+U 1 1 6197A54B
+P 2850 6400
+F 0 "AD1" H 2900 6650 50  0000 L CNN
+F 1 "WS2812B" H 2850 6150 50  0000 L CNN
+F 2 "LED_SMD:LED_WS2812B_PLCC4_5.0x5.0mm_P3.2mm" H 2900 6100 50  0001 L TNN
+F 3 "https://cdn-shop.adafruit.com/datasheets/WS2812B.pdf" H 2950 6025 50  0001 L TNN
+	1    2850 6400
+	1    0    0    -1
+$EndComp
+$Comp
+L power:GND #PWR0136
+U 1 1 6197BC25
+P 2850 6850
+F 0 "#PWR0136" H 2850 6600 50  0001 C CNN
+F 1 "GND" H 2855 6677 50  0000 C CNN
+F 2 "" H 2850 6850 50  0001 C CNN
+F 3 "" H 2850 6850 50  0001 C CNN
+	1    2850 6850
+	1    0    0    -1
+$EndComp
+Wire Wire Line
+	2850 6700 2850 6800
+$Comp
+L power:+5V #PWR0137
+U 1 1 61982203
+P 2850 6000
+F 0 "#PWR0137" H 2850 5850 50  0001 C CNN
+F 1 "+5V" H 2865 6173 50  0000 C CNN
+F 2 "" H 2850 6000 50  0001 C CNN
+F 3 "" H 2850 6000 50  0001 C CNN
+	1    2850 6000
+	-1   0    0    -1
+$EndComp
+Wire Wire Line
+	2850 6000 2850 6050
+Text GLabel 1200 4800 0    50   Input ~ 0
+G23
+Text GLabel 2400 6400 0    50   Input ~ 0
+G23
+Wire Wire Line
+	2400 6400 2550 6400
+$Comp
+L Device:C_Small C1
+U 1 1 6198D6DD
+P 3400 6400
+F 0 "C1" H 3492 6446 50  0000 L CNN
+F 1 "10pF" H 3492 6355 50  0000 L CNN
+F 2 "Capacitor_THT:C_Disc_D5.0mm_W2.5mm_P5.00mm" H 3400 6400 50  0001 C CNN
+F 3 "~" H 3400 6400 50  0001 C CNN
+	1    3400 6400
+	1    0    0    -1
+$EndComp
+Wire Wire Line
+	3400 6300 3400 6050
+Wire Wire Line
+	3400 6050 2850 6050
+Connection ~ 2850 6050
+Wire Wire Line
+	2850 6050 2850 6100
+Wire Wire Line
+	3400 6500 3400 6800
+Wire Wire Line
+	3400 6800 2850 6800
+Connection ~ 2850 6800
+Wire Wire Line
+	2850 6800 2850 6850
+Wire Notes Line
+	3800 5750 3800 7100
+Wire Notes Line
+	700  5750 3800 5750
+Wire Notes Line
+	700  7100 3800 7100
 $EndSCHEMATC

Commit message: pcb minor changes
Parts:
- renumbered temp1 to HT1, temp2 to HT2, temp6 to HT6
Changed lines of the file:
@@
 	8600 2750 9000 2750
 $Comp
-L Connector_Generic_MountingPin:Conn_01x03_MountingPin temp1
+L Connector_Generic_MountingPin:Conn_01x03_MountingPin HT1
 U 1 1 619D5390
 P 4950 2100
-F 0 "temp1" H 4900 2300 50  0000 L CNN
+F 0 "HT1" H 4900 2300 50  0000 L CNN
 F 1 "4" H 5000 2100 50  0000 L CNN
 F 2 "Connector_JST:JST_XH_B3B-XH-AM_1x03_P2.50mm_Vertical" H 4950 2100 50  0001 C CNN
@@
 $EndComp
 $Comp
-L Connector_Generic_MountingPin:Conn_01x03_MountingPin temp2
+L Connector_Generic_MountingPin:Conn_01x03_MountingPin HT2
 U 1 1 619D2951
 P 4250 2100
-F 0 "temp2" H 4200 2300 50  0000 L CNN
+F 0 "HT2" H 4200 2300 50  0000 L CNN
 F 1 "4" H 4300 2100 50  0000 L CNN
 F 2 "Connector_JST:JST_XH_B3B-XH-AM_1x03_P2.50mm_Vertical" H 4250 2100 50  0001 C CNN
@@
 $EndComp
 $Comp
-L Connector_Generic_MountingPin:Conn_01x03_MountingPin temp6
+L Connector_Generic_MountingPin:Conn_01x03_MountingPin HT6
 U 1 1 618718D1
 P 3550 2100
-F 0 "temp6" H 3500 2300 50  0000 L CNN
+F 0 "HT6" H 3500 2300 50  0000 L CNN
 F 1 "4" H 3600 2100 50  0000 L CNN
 F 2 "Connector_JST:JST_XH_B3B-XH-AM_1x03_P2.50mm_Vertical" H 3550 2100 50  0001 C CNN
